Commit message: Completed ragdoll test

File: legs.urdf (robot description, URDF)
Before this commit: robot legs, 13 links, 12 joints
Links:
- link base_link: mass None -> 10; geometry collision box size=0.2 0.4 0.8; visual box size=0.2 0.4 0.8
- link left_ankle: mass None -> 0.1; geometry collision sphere radius=0.1; visual sphere radius=0.1
- link left_foot: mass None -> 2; geometry collision box size=0.3 0.1 0.15; visual box size=0.3 0.1 0.15
- link left_hip: mass None -> 0.1
- link left_knee: mass None -> 0.1
- link left_shin: mass None -> 5; geometry collision box size=0.2 0.1 0.4; visual box size=0.2 0.1 0.4
- link left_thigh: mass None -> 8; geometry collision box size=0.2 0.1 0.4; visual box size=0.2 0.1 0.4
- link right_ankle: mass None -> 0.1; geometry collision sphere radius=0.1; visual sphere radius=0.1
- link right_foot: mass None -> 2; geometry collision box size=0.3 0.1 0.15; visual box size=0.3 0.1 0.15
- link right_hip: mass None -> 0.1
- link right_knee: mass None -> 0.1; geometry collision sphere radius=0.1; visual sphere radius=0.1
- link right_shin: mass None -> 5; geometry collision box size=0.2 0.1 0.4; visual box size=0.2 0.1 0.4
- link right_thigh: mass None -> 8; geometry collision box size=0.2 0.1 0.4; visual box size=0.2 0.1 0.4
Joints:
- removed joint base_to_left_thigh
- removed joint base_to_right_thigh
- added joint left_hip_to_left_thigh: type revolute, parent left_hip, child left_thigh, origin xyz=0 0 -0.2 rpy=0 0 0, axis 0 1 0, limit lower=-0.785398 upper=0.785398 effort=1000.0 velocity=0.5
- added joint right_hip_to_right_knee: type revolute, parent right_hip, child right_thigh, origin xyz=0 0 -0.2 rpy=0 0 0, axis 0 1 0, limit lower=-0.785398 upper=0.785398 effort=1000.0 velocity=0.5
- joint base_to_left_hip: axis 0 1 0 -> (none); origin xyz=0 -0.15 1.1 -> xyz=0 -0.1 -0.4; type continuous -> fixed
- joint base_to_right_hip: axis 0 1 0 -> (none); origin xyz=0 0.15 1.1 -> xyz=0 0.1 -0.4; type continuous -> fixed
- joint left_ankle_to_left_foot: limit (none) -> lower=0 upper=0.349066 effort=1000.0 velocity=0.5; origin xyz=0.15 0 0 -> xyz=0.15 0 0 rpy=0 0 0; type continuous -> revolute
- joint left_knee_to_left_shin: limit (none) -> lower=0 upper=1.5708 effort=1000.0 velocity=0.5; origin xyz=0 0 -0.25 -> xyz=0 0 -0.2 rpy=0 0 0; type continuous -> revolute
- joint left_shin_to_left_ankle: axis 0 1 0 -> (none); type continuous -> fixed
- joint left_thigh_to_left_knee: axis 0 1 0 -> (none); type continuous -> fixed
- joint right_ankle_to_right_foot: axis (none) -> 0 1 0; limit (none) -> lower=0 upper=0.349066 effort=1000.0 velocity=0.5; origin xyz=0.15 0 0 -> xyz=0.15 0 0 rpy=0 0 0; type fixed -> revolute
- joint right_knee_to_right_shin: limit (none) -> lower=0 upper=1.5708 effort=1000.0 velocity=0.5; origin xyz=0 0 -0.25 -> xyz=0 0 -0.2 rpy=0 0 0; type continuous -> revolute
- joint right_shin_to_right_ankle: axis 0 1 0 -> (none); type continuous -> fixed
- joint right_thigh_to_right_knee: type continuous -> fixed

Commit message: Fixed joint origins so joints hinge around correct point, giving more natural looking movement

File: legs.urdf (robot description, URDF)
Before this commit: robot legs, 13 links, 12 joints
Links:
- link left_knee: geometry collision sphere radius=0.1; visual sphere radius=0.1
- link right_knee: geometry visual sphere radius=0.1
Joints:
- removed joint right_hip_to_right_knee
- added joint right_hip_to_right_thigh: type revolute, parent right_hip, child right_thigh, origin xyz=0 0 0 rpy=0 0 0, axis 0 1 0, limit lower=-0.785398 upper=0.785398 effort=1000.0 velocity=0.5
- joint base_to_left_hip: origin xyz=0 -0.1 -0.4 -> xyz=0 0.15 -0.4
- joint base_to_right_hip: origin xyz=0 0.1 -0.4 -> xyz=0 -0.15 -0.4
- joint left_ankle_to_left_foot: limit lower=0 upper=0.349066 effort=1000.0 velocity=0.5 -> lower=-0.436332 upper=0.610865 effort=1000.0 velocity=0.5; origin xyz=0.15 0 0 rpy=0 0 0 -> xyz=0 0 0 rpy=0 0 0
- joint left_hip_to_left_thigh: origin xyz=0 0 -0.2 rpy=0 0 0 -> xyz=0 0 0 rpy=0 0 0
- joint left_knee_to_left_shin: origin xyz=0 0 -0.2 rpy=0 0 0 -> xyz=0 0 0 rpy=0 0 0
- joint left_shin_to_left_ankle: origin xyz=0 0 -0.2 -> xyz=0 0 -0.4
- joint left_thigh_to_left_knee: axis (none) -> 0 1 0; origin xyz=0 0 -0.2 -> xyz=0 0 -0.4
- joint right_ankle_to_right_foot: limit lower=0 upper=0.349066 effort=1000.0 velocity=0.5 -> lower=-0.436332 upper=0.610865 effort=1000.0 velocity=0.5; origin xyz=0.15 0 0 rpy=0 0 0 -> xyz=0 0 0 rpy=0 0 0
- joint right_knee_to_right_shin: origin xyz=0 0 -0.2 rpy=0 0 0 -> xyz=0 0 0 rpy=0 0 0
- joint right_shin_to_right_ankle: origin xyz=0 0 -0.2 -> xyz=0 0 -0.4
- joint right_thigh_to_right_knee: axis 0 1 0 -> (none); origin xyz=0 0 -0.2 -> xyz=0 0 -0.4
